File: 808_bass_drum.sch (EAGLE design)
At the start: 56 parts, among them IC1 TL072P, Q1 2N3906, Q10 2N3904, Q11 2N3904, Q7 2N3904, Q8 2N3904, Q9 2N3904

Commit message: 93pct ar
Parts:
- added C1, C2: 10u, rcl:CPOL-USB45181A
- added C4, C5: 100n, rcl:C-US050-024X044
- added U$1, U$3: FB, adafruit:FB
- C38, C45: device TR808clone:C-EU075-032X103 -> TR808clone:C-EU050-030X075
- C39: device TR808clone:C-EU050-024X044 -> TR808clone:C-EU050-025X075
- C48: device TR808clone:C-EU025-025X050 -> TR808clone:C-EU050-025X075
- R156, R159, R160, R161, R165, R167, R168, R169, R171, R174, R177: device TR808clone:R-EU_0207/5V -> TR808clone:R-EU_0207/7
- R166, R173, R175, R176: device TR808clone:R-EU_0207/5V -> TR808clone:R-EU_0309/10
Connections:
- new net N$5: U$1.1, U$2.+12V
- new net N$6: U$2.-12V, U$3.1
- net +12V: now also C1.+, C4.1, U$1.2; no longer U$2.+12V
- net -12V: now also C2.-, C5.2, U$3.2; no longer U$2.-12V
- net GND: now also C1.-, C2.+, C4.2, C5.1
Other:
- moved on the sheet: ACCENT, TRIG, U$2

Commit message: routed
Parts:
- removed R165: 47K, TR808clone:R-EU_0207/7
- R173, R175: device TR808clone:R-EU_0309/10 -> TR808clone:R-EU_0207/7
- R177: device TR808clone:R-EU_0207/7 -> TR808clone:R-EU_0309/10
Connections:
- net GND: no longer R165.2
- net N$168: no longer R165.1
Changed lines of the file:
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@@
 <part name="V104" library="supply1" deviceset="GND" device=""/>
 <part name="R166" library="TR808clone" deviceset="R-EU_" device="0309/10" value="6K8"/>
-<part name="R165" library="TR808clone" deviceset="R-EU_" device="0207/7" value="47K"/>
-<part name="V105" library="supply1" deviceset="GND" device=""/>
 <part name="C42" library="TR808clone" deviceset="C-EU" device="050-024X044" value="15n"/>
 <part name="C41" library="TR808clone" deviceset="C-EU" device="050-024X044" value="15n"/>
@@
 <part name="R172" library="TR808clone" deviceset="R-EU_" device="0207/5V" value="10K"/>
 <part name="V110" library="supply1" deviceset="GND" device=""/>
-<part name="R177" library="TR808clone" deviceset="R-EU_" device="0207/7" value="82K"/>
+<part name="R177" library="TR808clone" deviceset="R-EU_" device="0309/10" value="82K"/>
 <part name="R176" library="TR808clone" deviceset="R-EU_" device="0309/10" value="100K"/>
 <part name="C48" library="TR808clone" deviceset="C-EU" device="050-025X075" value="220p"/>
-<part name="R173" library="TR808clone" deviceset="R-EU_" device="0309/10" value="6K8"/>
+<part name="R173" library="TR808clone" deviceset="R-EU_" device="0207/7" value="6K8"/>
 <part name="V111" library="supply1" deviceset="GND" device=""/>
 <part name="V112" library="supply1" deviceset="GND" device=""/>
 <part name="R174" library="TR808clone" deviceset="R-EU_" device="0207/7" value="100K"/>
-<part name="R175" library="TR808clone" deviceset="R-EU_" device="0309/10" value="1K"/>
+<part name="R175" library="TR808clone" deviceset="R-EU_" device="0207/7" value="1K"/>
 <part name="C49" library="TR808clone" deviceset="CPOL-EU" device="E2.5-5" value=".47/50"/>
 <part name="C43" library="TR808clone" deviceset="CPOL-EU" device="E2.5-5" value="33/6.3"/>
@@
 <instance part="V104" gate="1" x="60.96" y="48.26"/>
 <instance part="R166" gate="G$1" x="68.58" y="71.12" rot="R90"/>
-<instance part="R165" gate="G$1" x="68.58" y="58.42" rot="R270"/>
-<instance part="V105" gate="1" x="68.58" y="48.26"/>
 <instance part="C42" gate="G$1" x="81.28" y="76.2" rot="R90"/>
 <instance part="C41" gate="G$1" x="58.42" y="76.2" rot="R90"/>
@@
 </segment>
 <segment>
-<pinref part="R165" gate="G$1" pin="2"/>
-<pinref part="V105" gate="1" pin="GND"/>
-<wire x1="68.58" y1="50.8" x2="68.58" y2="53.34" width="0.1524" layer="91"/>
-</segment>
-<segment>
 <pinref part="R168" gate="G$1" pin="2"/>
 <pinref part="V108" gate="1" pin="GND"/>
@@
 <wire x1="60.96" y1="66.04" x2="68.58" y2="66.04" width="0.1524" layer="91"/>
 <pinref part="R166" gate="G$1" pin="1"/>
-<pinref part="R165" gate="G$1" pin="1"/>
-<wire x1="68.58" y1="63.5" x2="68.58" y2="66.04" width="0.1524" layer="91"/>
 <junction x="68.58" y="66.04"/>
 <wire x1="60.96" y1="63.5" x2="60.96" y2="66.04" width="0.1524" layer="91"/>

Commit message: cutout
Parts:
- C38, C45: device TR808clone:C-EU050-030X075 -> TR808clone:C-EU050-024X044
- C39: device TR808clone:C-EU050-025X075 -> TR808clone:C-EU050-024X044
- R163: device TR808clone:R-EU_0207/5V -> TR808clone:R-EU_0207/2V
Changed lines of the file:
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@@
 <part name="V85" library="supply1" deviceset="GND" device=""/>
 <part name="R156" library="TR808clone" deviceset="R-EU_" device="0207/7" value="1M"/>
-<part name="C38" library="TR808clone" deviceset="C-EU" device="050-030X075" value="100n"/>
+<part name="C38" library="TR808clone" deviceset="C-EU" device="050-024X044" value="100n"/>
 <part name="R155" library="TR808clone" deviceset="R-EU_" device="0207/5V" value="4K7"/>
 <part name="R154" library="TR808clone" deviceset="R-EU_" device="0207/5V" value="10K"/>
@@
 <part name="V101" library="supply1" deviceset="GND" device=""/>
 <part name="C40" library="TR808clone" deviceset="C-EU" device="050-024X044" value="15n"/>
-<part name="R163" library="TR808clone" deviceset="R-EU_" device="0207/5V" value="100K"/>
-<part name="C39" library="TR808clone" deviceset="C-EU" device="050-025X075" value="33n"/>
+<part name="R163" library="TR808clone" deviceset="R-EU_" device="0207/2V" value="100K"/>
+<part name="C39" library="TR808clone" deviceset="C-EU" device="050-024X044" value="33n"/>
 <part name="R159" library="TR808clone" deviceset="R-EU_" device="0207/7" value="100K"/>
 <part name="D52" library="TR808clone" deviceset="1N4148" device="DO35-7"/>
@@
 <part name="R168" library="TR808clone" deviceset="R-EU_" device="0207/7" value="22K"/>
 <part name="V108" library="supply1" deviceset="GND" device=""/>
-<part name="C45" library="TR808clone" deviceset="C-EU" device="050-030X075" value="100n"/>
+<part name="C45" library="TR808clone" deviceset="C-EU" device="050-024X044" value="100n"/>
 <part name="V109" library="supply1" deviceset="GND" device=""/>
 <part name="R172" library="TR808clone" deviceset="R-EU_" device="0207/5V" value="10K"/>
