File: 808_bass_drum.brd (EAGLE design)
At the start: 100 x 80 mm, 56 parts, among them IC1 TL072P, Q1 2N3906, Q10 2N3904, Q11 2N3904, Q7 2N3904, Q8 2N3904, Q9 2N3904

Commit message: 93pct ar
Parts:
- added C1, C2: 10u, rcl:B45181A
- added C4, C5: 100n, rcl:C050-024X044
- added U$1, U$3: FB, adafruit:FB
- C38, C45: device TR808clone:C075-032X103 -> TR808clone:C050-030X075
- C39: device TR808clone:C050-024X044 -> TR808clone:C050-025X075
- C48: device TR808clone:C025-025X050 -> TR808clone:C050-025X075
- R156, R159, R160, R161, R165, R167, R168, R169, R171, R174, R177: device TR808clone:0207/5V -> TR808clone:0207/7
- R166, R173, R175, R176: device TR808clone:0207/5V -> TR808clone:0309/10
- moved TUNE_MOD 43.2 mm to (53.3, 3.81)
- moved R174 35.6 mm to (74.9, 22.9)
- moved R172 31.1 mm to (34.3, 10.2), turned to 180 degrees
- moved R173 30.2 mm to (35.6, 39.4), turned to 180 degrees
- moved C40 29.6 mm to (55.9, 53.3)
- moved R159 28.5 mm to (68.6, 21.6)
- moved Q7 26.9 mm to (61.0, 12.7)
- moved R163 23.4 mm to (49.5, 49.5), turned to 270 degrees
- moved Q11 23.0 mm to (73.7, 49.5), turned to 0 degrees
- moved R160 23.0 mm to (73.7, 44.5), turned to 180 degrees
- moved R162 23.0 mm to (57.1, 48.3)
- moved C42 22.9 mm to (43.2, 44.5), turned to 0 degrees
- moved Q10 22.2 mm to (64.8, 54.6)
- moved TONE 21.6 mm to (31.8, 3.81)
- moved DECAY 21.6 mm to (10.2, 3.81)
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Connections:
- new net N$5: U$1.P$1, U$2.10, U$2.9
- new net N$6: U$2.1, U$2.2, U$3.P$1
- net +12V: now also C1.+, C4.1, U$1.P$2; no longer U$2.10, U$2.9
- net -12V: now also C2.-, C5.2, U$3.P$2; no longer U$2.1, U$2.2
- net GND: now also C1.-, C2.+, C4.2, C5.1

Commit message: routed
Parts:
- removed R165: 47K, TR808clone:0207/7
- R173, R175: device TR808clone:0309/10 -> TR808clone:0207/7
- R177: device TR808clone:0207/7 -> TR808clone:0309/10
- moved R174 9.92 mm to (82.5, 29.2), turned to 180 degrees
- moved C42 8.03 mm to (45.7, 36.8), turned to 270 degrees
- moved C39 6.75 mm to (72.4, 26.0), turned to 180 degrees
- moved D52 6.35 mm to (80.0, 38.1)
- moved C48 5.12 mm to (53.3, 36.2)
- moved R161 4.49 mm to (69.2, 34.9)
- moved R159 2.84 mm to (69.8, 19.1), turned to 0 degrees
- moved C41 2.54 mm to (38.1, 45.7)
- moved R175 1.80 mm to (88.9, 24.1)
- moved Q7 1.80 mm to (62.2, 14.0)
- moved C40 1.42 mm to (55.2, 52.1)
- moved C50 1.42 mm to (50.8, 31.1), turned to 90 degrees
- moved D53 1.27 mm to (52.1, 43.2)
- moved Q10 1.27 mm to (64.8, 55.9)
- moved R176 1.27 mm to (50.8, 21.6)
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Connections:
- net GND: no longer R165.2
- net N$168: no longer R165.1
Routing:
- net GND: track 0.00 -> 488.1 mm
- net +12V: track 0.00 -> 116.1 mm
- net N$198: track 0.00 -> 100.5 mm
- net N$202: track 0.00 -> 64.1 mm
- net -12V: track 0.00 -> 63.4 mm
- net N$195: track 0.00 -> 61.8 mm
- net N$205: track 0.00 -> 56.1 mm, vias 0 -> 2
- net N$192: track 0.00 -> 48.3 mm
- net N$1: track 0.00 -> 45.5 mm
- net N$197: track 0.00 -> 42.2 mm
- net N$168: track 0.00 -> 35.2 mm
- net N$190: track 0.00 -> 33.0 mm
- net TRIG: track 0.00 -> 27.6 mm
- net N$204: track 0.00 -> 25.9 mm
- net N$4: track 0.00 -> 22.2 mm
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
Commit message: cutout
Parts:
- C38, C45: device TR808clone:C050-030X075 -> TR808clone:C050-024X044
- C39: device TR808clone:C050-025X075 -> TR808clone:C050-024X044
- R163: device TR808clone:0207/5V -> TR808clone:0207/2V
- moved TRIG 10.9 mm to (17.8, 61.0)
- moved C50 9.55 mm to (51.4, 40.6), turned to 0 degrees
- moved D53 2.84 mm to (53.3, 45.7)
- moved R163 1.80 mm to (50.8, 50.8)
- moved R159 1.27 mm to (71.1, 19.1)
- moved C39 1.27 mm to (72.4, 27.3)
- moved C45 1.27 mm to (82.5, 20.3)
- moved R174 1.27 mm to (82.5, 30.5), turned to 270 degrees
- moved C49 1.27 mm to (72.4, 14.0)
- moved C48 1.27 mm to (54.1, 35.2)
- moved C40 1.05 mm to (56.3, 52.3)
- moved R166 0.76 mm to (60.2, 38.1)
Routing:
- net N$205: track 56.1 -> 47.4 mm
- net GND: track 488.1 -> 480.9 mm
- net N$4: track 22.2 -> 16.8 mm
- net N$204: track 25.9 -> 30.4 mm
- net N$198: track 100.5 -> 99.3 mm
- net N$3: track 13.9 -> 12.7 mm
- net N$192: track 48.3 -> 49.1 mm
- net N$195: track 61.8 -> 62.5 mm
- net +12V: track 116.1 -> 116.7 mm
- net N$191: track 21.0 -> 21.6 mm
Other:
- board size 100 x 80 mm -> 101.3 x 81 mm

Commit message: working with tune and decay mods
Routing:
- net N$4: track 16.8 -> 15.5 mm
- net GND: track 480.9 -> 482.0 mm
- net C49: track 14.2 -> 15.0 mm
Changed lines of the file:
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@@
 <?xml version="1.0" encoding="utf-8"?>
 <!DOCTYPE eagle SYSTEM "eagle.dtd">
-<eagle version="7.2.0">
+<eagle version="7.1.0">
 <drawing>
 <settings>
@@
 <contactref element="R177" pad="2"/>
 <contactref element="C49" pad="-"/>
-<wire x1="71.628" y1="21.59" x2="64.77" y2="25.4" width="0.8128" layer="16"/>
-<wire x1="72.39" y1="15.24" x2="71.628" y2="21.59" width="0.8128" layer="16"/>
+<wire x1="71.628" y1="22.86" x2="64.77" y2="25.4" width="0.8128" layer="16"/>
+<wire x1="72.39" y1="15.24" x2="71.628" y2="22.86" width="0.8128" layer="16"/>
 </signal>
 <signal name="N$208">
@@
 <wire x1="69.93" y1="3.81" x2="69.93" y2="3.73" width="1.016" layer="16"/>
 <wire x1="69.93" y1="3.81" x2="69.93" y2="18.335" width="1.016" layer="16"/>
-<wire x1="69.93" y1="18.335" x2="69.977" y2="20.066" width="1.016" layer="16"/>
-<wire x1="69.977" y1="20.066" x2="62.357" y2="21.844" width="1.016" layer="16"/>
+<wire x1="69.93" y1="18.335" x2="69.977" y2="21.336" width="1.016" layer="16"/>
+<wire x1="69.977" y1="21.336" x2="62.357" y2="21.844" width="1.016" layer="16"/>
 <wire x1="92.79" y1="2.5" x2="86.44" y2="2.46" width="1.016" layer="16"/>
 <wire x1="86.44" y1="2.46" x2="86.36" y2="13.97" width="1.016" layer="16"/>
@@
 <contactref element="U$2" pad="16"/>
 <wire x1="11.43" y1="57.15" x2="8.89" y2="57.15" width="0.8128" layer="16"/>
-<wire x1="24.13" y1="60.96" x2="22.86" y2="60.96" width="0.8128" layer="16"/>
 <wire x1="13.97" y1="57.15" x2="11.43" y2="57.15" width="0.8128" layer="16"/>
 <wire x1="17.78" y1="60.96" x2="13.97" y2="57.15" width="0.8128" layer="16"/>
